File: doc/eagle/projects/quadcopter/motorcontrol.sch (EAGLE design)
At the start: 10 parts, among them IC1 MEGA8-P, Q1 8Mhz, X1 87758-0616

Commit message: Update circuit
Parts:
- removed X1: 87758-0616, con-molex:87758-0616
- added C10, C4, C6, C8: 100uF, rcl:C-EU025-025X050
- added C3, C5, C7, C9: 100uF, rcl:CPOL-EUE2-5
- added D1, D2, D3, D5: (no value), diode:SCHOTTKY-DIODEDO201T15
- added Q2, Q3, Q4, Q6: IRLZ44Z, transistor-power:IRLZ44Z
- added SV1: (no value), con-lstb:MA03-2
- added X2, X3, X4, X6: (no value), con-wago-500:W237-102
- renumbered IC2 to TS2940
Connections:
- new net M1GND: D5.A, Q4.D, X2-2.KL
- new net M2GND: D1.A, Q6.D, X6-2.KL
- new net M3GND: D2.A, Q2.D, X3-2.KL
- new net M4GND: D3.A, Q3.D, X4-2.KL
- new net PWM1: IC1.PD7(AIN1), Q4.G
- new net PWM2: IC1.PB0(ICP), Q6.G
- new net PWM3: IC1.PB1(OC1A), Q2.G
- new net PWM4: IC1.PB2(SS/OC1B), Q3.G
- net 3V3: now also IC1.AVCC, SV1.5; no longer X1-5.S
- net 3V7: now also C10.1, C3.+, C4.1, C5.+, C6.1, C7.+, C8.1, C9.+, D1.C, D2.C, D3.C, D5.C, X2-1.KL, X3-1.KL, X4-1.KL, X6-1.KL
- net GND: now also C10.2, C3.-, C4.2, C5.-, C6.2, C7.-, C8.2, C9.-, IC1.GND, Q2.S, Q3.S, Q4.S, Q6.S, SV1.1; no longer X1-1.S
- net MISO: now also SV1.6; no longer X1-6.S
- net MOSI: now also SV1.3; no longer X1-3.S
- net RESET: now also SV1.2; no longer X1-2.S
- net SCK: now also SV1.4; no longer X1-4.S
