File: doc/eagle/projects/quadcopter/motorcontrol.brd (EAGLE design)
At the start: 98.7 x 80 mm, 30 parts, among them IC1 MEGA8-P, Q1 8Mhz, Q2 IRLZ44Z, Q3 IRLZ44Z, Q4 IRLZ44Z, Q6 IRLZ44Z

Commit message: PCB producable
Parts:
- moved C10 22.9 mm to (5.08, 66.0), turned to 180 degrees
- moved C9 17.7 mm to (11.4, 66.0)
- moved C4 16.9 mm to (7.62, 26.7)
- moved C3 16.6 mm to (7.62, 21.6)
- moved C5 14.5 mm to (88.9, 15.2), turned to 270 degrees
- moved C6 8.52 mm to (83.8, 15.2), turned to 270 degrees
- moved C8 7.73 mm to (80.0, 68.6), turned to 180 degrees
- moved D1 5.24 mm to (86.4, 22.9)
- moved D2 1.80 mm to (86.4, 63.5)
- moved C7 1.80 mm to (80.0, 73.7), turned to 180 degrees
- moved Q6 1.27 mm to (82.5, 34.3)
Routing:
- net 3V7: track 167.2 -> 379.5 mm
- net M2GND: track 0.00 -> 41.4 mm
- net M3GND: track 0.00 -> 36.0 mm
- net PWM3: track 0.00 -> 29.7 mm
- net PWM2: track 0.00 -> 22.6 mm
- net 3V3: track 109.1 -> 112.6 mm
- net MOSI: track 28.3 -> 26.1 mm
